File: eagle/morse_lora_v1.sch (EAGLE design)
At the start: 20 parts

Commit message: draft layout
Parts:
- LEFT, OK, RIGHT: value (none) -> MOMENTARY-SWITCH-SPST-PTH-6.0MM; device adafruit:SWITCH_PUSHBUTTONEVQ-PE -> SparkFun-Switches:MOMENTARY-SWITCH-SPST-PTH-6.0MM
- MAIN: value (none) -> MOMENTARY-SWITCH-SPST-PTH-12MM; device adafruit:SWITCH_PUSHBUTTONEVQ-PE -> SparkFun-Switches:MOMENTARY-SWITCH-SPST-PTH-12MM
Connections:
- net N$12 renamed 35
- removed net 3V3@1: ESP32LORA.3V3@1, R1.2, R3.2
- removed net N$1: C1.2, D-BUT.C, R2.1
- removed net N$10: R2.2
- removed net N$11: R4.2
- removed net N$2: C3.1, ESP32LORA.39, R4.1, RIGHT.P$1
- removed net N$3: C2.2, ESP32LORA.34, LEFT.P$1, R3.1
- removed net N$7: C4.2, ESP32LORA.23, OK.P$1, R1.1
- removed net N$8: ESP32LORA.36, MAIN.P$1
- removed net N$9: D-BUT.A
- new net 23: C4.2, ESP32LORA.23, OK.2, R1.1
- new net 34: C2.2, ESP32LORA.34, LEFT.1, R3.1
- new net 36: C1.2, D-BUT.C, ESP32LORA.36, MAIN.1, R2.1
- new net 39: C3.1, ESP32LORA.39, R4.1, RIGHT.1
- net 3V3: now also D-BUT.A, ESP32LORA.3V3@1, R1.2, R2.2, R3.2, R4.2
- net GND: now also LEFT.2, MAIN.2, OK.1, RIGHT.2; no longer LEFT.P$2, MAIN.P$2, OK.P$2, RIGHT.P$2
Other:
- moved on the sheet: BUZZER, C2, C3, D-BLU, D-BUT, D-REC, R2, R3, R4, SLEEP

Commit message: draft layout
Changed lines of the file:
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@@
 <junction x="-129.54" y="177.8"/>
 <junction x="-139.7" y="177.8"/>
+<label x="-139.7" y="177.8" size="1.778" layer="95"/>
 </segment>
 </net>

Commit message: update pcb v1
Parts:
- SLEEP: value SWS001 -> (none); device smd-special:SWS001 -> adafruit:EG1218S
Connections:
- net 3V3: now also SLEEP.O
- net GND: now also ESP32LORA.GND@1, SLEEP.S; no longer SLEEP.1
- net N$13: now also SLEEP.P; no longer SLEEP.2
Changed lines of the file:
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@@
 <part name="R5" library="SparkFun-Resistors" deviceset="10KOHM" device="-HORIZ_KIT-1/4W-1%" value="10k"/>
 <part name="R6" library="SparkFun-Resistors" deviceset="10KOHM" device="-HORIZ_KIT-1/4W-1%" value="10k"/>
-<part name="SLEEP" library="smd-special" library_urn="urn:adsk.eagle:library:362" deviceset="SWS001" device="" package3d_urn="urn:adsk.eagle:package:26467/1"/>
 <part name="GND3" library="SparkFun-PowerSymbols" deviceset="GND" device=""/>
 <part name="LEFT" library="SparkFun-Switches" deviceset="MOMENTARY-SWITCH-SPST" device="-PTH-6.0MM"/>
@@
 <part name="OK" library="SparkFun-Switches" deviceset="MOMENTARY-SWITCH-SPST" device="-PTH-6.0MM"/>
 <part name="MAIN" library="SparkFun-Switches" deviceset="MOMENTARY-SWITCH-SPST" device="-PTH-12MM"/>
+<part name="SLEEP" library="adafruit" library_urn="urn:adsk.eagle:library:420" deviceset="EG1218" device="S" package3d_urn="urn:adsk.eagle:package:6240649/1"/>
 </parts>
 <sheets>
@@
 <attribute name="VALUE" x="-109.22" y="150.876" size="1.778" layer="96" font="vector" align="top-center"/>
 </instance>
-<instance part="SLEEP" gate="G$1" x="-132.08" y="147.32" smashed="yes" rot="R90">
-<attribute name="NAME" x="-129.54" y="144.78" size="1.778" layer="95" rot="R180"/>
-<attribute name="VALUE" x="-129.54" y="151.765" size="1.778" layer="96" rot="R180"/>
-</instance>
-<instance part="GND3" gate="1" x="-121.92" y="147.32" smashed="yes" rot="R90">
-<attribute name="VALUE" x="-120.396" y="147.32" size="1.778" layer="96" rot="R90" align="top-center"/>
+<instance part="GND3" gate="1" x="-121.92" y="144.78" smashed="yes" rot="R90">
+<attribute name="VALUE" x="-120.396" y="144.78" size="1.778" layer="96" rot="R90" align="top-center"/>
 </instance>
 <instance part="LEFT" gate="G$1" x="-88.9" y="160.02" smashed="yes">
@@
 <attribute name="NAME" x="-129.54" y="171.704" size="1.778" layer="95" font="vector" align="bottom-center"/>
 <attribute name="VALUE" x="-129.54" y="169.672" size="1.778" layer="96" font="vector" align="top-center"/>
+</instance>
+<instance part="SLEEP" gate="1" x="-134.62" y="147.32" smashed="yes" rot="R270">
+<attribute name="NAME" x="-136.525" y="153.67" size="1.778" layer="95"/>
+<attribute name="VALUE" x="-131.445" y="151.13" size="1.778" layer="96"/>
 </instance>
 </instances>
@@
 </segment>
 <segment>
+<pinref part="GND3" gate="1" pin="GND"/>
+<wire x1="-129.54" y1="142.24" x2="-124.46" y2="144.78" width="0.1524" layer="91"/>
+<pinref part="SLEEP" gate="1" pin="S"/>
+</segment>
+<segment>
+<pinref part="ESP32LORA" gate="G$1" pin="GND@1"/>
+<wire x1="-175.26" y1="177.8" x2="-190.5" y2="177.8" width="0.1524" layer="91"/>
 <pinref part="GND6" gate="1" pin="GND"/>
 <wire x1="-180.34" y1="139.7" x2="-180.34" y2="134.62" width="0.1524" layer="91"/>
@@
 <pinref part="OK" gate="G$1" pin="1"/>
 <junction x="-180.34" y="139.7"/>
-</segment>
-<segment>
+<wire x1="-190.5" y1="177.8" x2="-190.5" y2="134.62" width="0.1524" layer="91"/>
+<wire x1="-190.5" y1="134.62" x2="-180.34" y2="134.62" width="0.1524" layer="91"/>
+<junction x="-180.34" y="134.62"/>
+<wire x1="-180.34" y1="134.62" x2="-180.34" y2="121.92" width="0.1524" layer="91"/>
+<wire x1="-180.34" y1="121.92" x2="-106.68" y2="121.92" width="0.1524" layer="91"/>
+<wire x1="-106.68" y1="121.92" x2="-106.68" y2="134.62" width="0.1524" layer="91"/>
 <pinref part="GND2" gate="1" pin="GND"/>
 <pinref part="BUZZER" gate="G$1" pin="2"/>
 <wire x1="-111.76" y1="134.62" x2="-119.38" y2="134.62" width="0.1524" layer="91"/>
-</segment>
-<segment>
-<pinref part="SLEEP" gate="G$1" pin="1"/>
-<pinref part="GND3" gate="1" pin="GND"/>
-<wire x1="-127" y1="147.32" x2="-124.46" y2="147.32" width="0.1524" layer="91"/>
+<wire x1="-106.68" y1="134.62" x2="-111.76" y2="134.62" width="0.1524" layer="91"/>
+<junction x="-111.76" y="134.62"/>
 </segment>
 </net>
@@
 </net>
 <net name="3V3" class="0">
-<segment>
-<pinref part="R6" gate="G$1" pin="1"/>
-<wire x1="-114.3" y1="152.4" x2="-116.84" y2="152.4" width="0.1524" layer="91"/>
-<junction x="-116.84" y="152.4"/>
-<label x="-118.11" y="153.67" size="1.778" layer="95"/>
-</segment>
 <segment>
 <pinref part="ESP32LORA" gate="G$1" pin="3V3@1"/>
@@
 <label x="-139.7" y="195.58" size="1.778" layer="95"/>
 </segment>
+<segment>
+<pinref part="R6" gate="G$1" pin="1"/>
+<label x="-118.11" y="153.67" size="1.778" layer="95"/>
+<pinref part="SLEEP" gate="1" pin="O"/>
+<wire x1="-129.54" y1="147.32" x2="-129.54" y2="152.4" width="0.1524" layer="91"/>
+<wire x1="-129.54" y1="152.4" x2="-114.3" y2="152.4" width="0.1524" layer="91"/>
+</segment>
 </net>
 <net name="36" class="0">
@@
 <wire x1="-129.54" y1="180.34" x2="-129.54" y2="177.8" width="0.1524" layer="91"/>
 <pinref part="D-BUT" gate="D1" pin="C"/>
-<junction x="-139.7" y="170.18"/>
 <wire x1="-139.7" y1="182.88" x2="-139.7" y2="177.8" width="0.1524" layer="91"/>
 <wire x1="-139.7" y1="177.8" x2="-139.7" y2="170.18" width="0.1524" layer="91"/>
@@
 <wire x1="-144.78" y1="152.4" x2="-142.24" y2="152.4" width="0.1524" layer="91"/>
 <wire x1="-142.24" y1="152.4" x2="-142.24" y2="147.32" width="0.1524" layer="91"/>
-<pinref part="SLEEP" gate="G$1" pin="2"/>
-<wire x1="-142.24" y1="147.32" x2="-139.7" y2="147.32" width="0.1524" layer="91"/>
-</segment>
-</net>
+<wire x1="-142.24" y1="147.32" x2="-139.7" y2="144.78" width="0.1524" layer="91"/>
+<pinref part="SLEEP" gate="1" pin="P"/>
+</segment>
+</net>
