File: eagle/morse_lora_v4.brd (EAGLE design)
At the start: 55 x 82.9 mm, 20 parts

Commit message: board v3 and v4
Routing:
- net 36: track 150.5 -> 146.3 mm
Changed lines of the file:
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@@
 <drawing>
 <settings>
-<setting alwaysvectorfont="yes"/>
+<setting alwaysvectorfont="no"/>
 <setting verticaltext="up"/>
 </settings>
@@
 <contactref element="R6" pad="P$2"/>
 <contactref element="ESP32LORA" pad="P$28"/>
-<wire x1="10.668" y1="62.103" x2="10.541" y2="61.976" width="0.1524" layer="1"/>
 <wire x1="14.097" y1="61.976" x2="14.097" y2="69.85" width="0.1524" layer="16"/>
 <wire x1="14.097" y1="69.85" x2="22.733" y2="69.85" width="0.1524" layer="16"/>
@@
 <contactref element="R2" pad="P$1"/>
 <contactref element="C1" pad="2"/>
-<wire x1="47.879" y1="55.626" x2="22.098" y2="55.626" width="0.1524" layer="1"/>
+<wire x1="47.879" y1="55.626" x2="24.511" y2="55.626" width="0.1524" layer="1"/>
+<wire x1="24.511" y1="55.626" x2="22.987" y2="55.626" width="0.1524" layer="1"/>
 <wire x1="22.987" y1="41.65599375" x2="17.907" y2="41.65599375" width="0.1524" layer="1"/>
-<wire x1="22.987" y1="41.65599375" x2="22.098" y2="41.65599375" width="0.1524" layer="1"/>
-<wire x1="24.5618" y1="57.8866" x2="22.098" y2="57.8866" width="0.1524" layer="1"/>
-<wire x1="22.098" y1="57.8866" x2="22.098" y2="55.626" width="0.1524" layer="1"/>
-<wire x1="22.098" y1="55.626" x2="22.098" y2="41.65599375" width="0.1524" layer="1"/>
+<wire x1="22.987" y1="41.65599375" x2="22.987" y2="55.626" width="0.1524" layer="1"/>
 <contactref element="D-BUT" pad="K"/>
 <contactref element="ESP32LORA" pad="P$33"/>
@@
 <wire x1="52.451" y1="96.647" x2="52.4818" y2="96.6162" width="0.1524" layer="1"/>
 <wire x1="52.4818" y1="96.6162" x2="52.4818" y2="60.452" width="0.1524" layer="1"/>
+<wire x1="24.5618" y1="57.8866" x2="24.5618" y2="56.261" width="0.1524" layer="1"/>
+<wire x1="24.5618" y1="56.261" x2="24.5618" y2="55.6768" width="0.1524" layer="1"/>
+<wire x1="24.5618" y1="55.6768" x2="24.511" y2="55.626" width="0.1524" layer="1"/>
 </signal>
 <signal name="N$13">
